File: hardware/vu_meter.sch (EAGLE design)
At the start: 90 parts, among them IC1 MCP604, IC2 MCP1700 3V3, IC3 MEGA88, IC4 MCP1700 2V5, IC5 MCP604, IC6 MCP604, Q2 BSS138, Q3 BSS138

Commit message: Updated schematic and added bill of materials
Parts:
- removed D1: BAT54C, diode:BAT54C
- removed IC4: MCP1700 2V5, linear:MCP1703CB
- added C30, C31, C32, C33: 22pF, rcl:C-EUC0805
- added U$1: MCP1525, SparkFun:MCP9700SMD
- C16: value 1uF* -> 100nF
- D2, D3: value BAV99 -> BAT54S
- R2, R3: value 100k -> 47k
Connections:
- net +5V: now also U$1.VCC; no longer D1.CC, IC4.VI
- net GND: now also U$1.GND; no longer IC4.GND
- net GND1: now also U$1.VO; no longer IC4.VO
- net N$19: now also C31.1; no longer D1.A2
- net N$25: now also C31.2
- net N$27: now also C30.2
- net N$29: now also C32.1
- net N$33: now also C33.1; no longer D1.A1
- net N$34: now also C33.2
- net N$36: now also C32.2
- net N$37: now also C30.1

Commit message: Updates to design & build process
Parts:
- removed C19, C25, C27: 100nF, rcl:C-EUC0805
- removed C20, C21, C22, C23: 220nF, rcl:C-EUC0805
- removed C24, C26, C28, C29: 2u2, rcl:C-EUC0805
- removed C30, C31, C32, C33: 22pF, rcl:C-EUC0805
- removed H1, H2, H3, H4: MOUNT-HOLE3.2, holes:MOUNT-HOLE3.2
- removed IC5, IC6: MCP604, linear:MCP604SL
- removed ISP: (no value), pinhead:PINHD-2X5
- removed L1, L2, L3: (no value), rcl:L-EUL3216C
- removed Q3: BSS138, transistor-small-signal:BSS123
- removed R32: 10k, rcl:R-EU_R0805
- removed R33, R34, R35, R36: 110k, rcl:R-EU_R0805
- removed U$1: MCP1525, SparkFun:MCP9700SMD
- added B1: ARDUINO_UNO_R3NO_HOLES, SparkFun-Boards:ARDUINO_UNO_R3NO_HOLES
- added IC4: MCP6002SN, linear:MCP602SN
- added JP3: (no value), pinhead:PINHD-1X4
- C11: value 22pF -> 330n
- C12, C13: value 100nF -> 330n
- C14: value 1uF* -> 330n
- C15: value 1uF* -> 47nF
- C16: value 100nF -> 47nF
- C17: value 1uF* -> 100nF
- C3: value 10nF -> 220nF
- C4: value 100nF -> 220nF
- C5: value 220nF -> 1uF*
- C6: value 220nF -> 100nF
- C7, C8: value 100nF -> 22pF
- C9: value 100uF -> 22pF; device rcl:CPOL-EUB/3528-21R -> rcl:C-EUC0805
- IC1: value MCP604 -> MCP1525; device linear:MCP604SL -> SparkFun:MCP9700SMD
- IC2: value MCP1700 3V3 -> MCP604; device linear:MCP1703CB -> linear:MCP604SL
- IC3: value MEGA88 -> MCP6004; device avr-7:MEGA48/88/168-AU -> linear:MCP604SL
- JP2: value MICRO_USB -> (none); device vu_meter:MICRO_USB -> pinhead:PINHD-2X2
- JP4: device pinhead:PINHD-2X4 -> pinhead:PINHD-1X4
- Q1: value (none) -> BSS138; device crystal:CRYSTALHC49S -> transistor-small-signal:BSS123
- R1: value 10k(A) -> 10k
- R12, R17: value 100k -> 10k
- R13, R16: value 220k -> 10k
- R14: value 100k -> 220k; device rcl:R-EU_R0805 -> rcl:R-EU_M0805
- R15: value 22k -> 220k; device rcl:R-EU_R0805 -> rcl:R-EU_M0805
- R18: value 22k -> 220k
- R19, R20, R21: value 100k -> 220k; device rcl:R-EU_M0805 -> rcl:R-EU_R0805
- R2, R3: value 47k -> 100k
- R22: value 100k -> 82k; device rcl:R-EU_M0805 -> rcl:R-EU_R0805
- R23: value 100 -> 82k
- R24: value 100 -> 220
- R25: value 1k -> 220
- R26: value 1k -> 30k; device rcl:R-EU_R0805 -> rcl:R-EU_M0805
- R27: value 10k -> 30k; device rcl:R-EU_R0805 -> rcl:R-EU_M0805
- R28: value 10k -> 1k
- R29: value 100k -> 1k; device rcl:R-EU_M0805 -> rcl:R-EU_R0805
- R30: value 100k -> 220k
- R31: value 10k -> 220k; device rcl:R-EU_R0805 -> rcl:R-EU_M0805
- R4: value 10k -> 100k
Connections:
- removed net N$12: D4.C, IC5A.-IN, R23.1
- removed net N$21: IC3.PB3(MOSI/OC2A/PCINT3), ISP.1
- removed net N$22: IC3.PB5(SCK/PCINT5), ISP.7
- removed net N$29: C32.1, IC1C.OUT, IC6A.+IN, R12.1, R18.2
- removed net N$30: C1.+, C2.1, C4.1, IC3.VCC@1, IC3.VCC@2, L1.1
- removed net N$32: C8.1, IC3.AVCC, L3.2
- removed net N$49: IC6B.-IN, R16.1, R17.1, R18.1, R20.2
- removed net N$5: C11.2, IC3.PB7(XTAL2/TOSC2/PCINT7), Q1.1
- removed net N$50: IC6B.OUT, R20.1, R22.2
- removed net N$51: C21.2, IC6C.+IN, R22.1
- removed net N$52: C23.2, IC6C.-IN, R30.1
- removed net N$53: C23.1, IC6C.OUT, R16.2, R34.2
- removed net N$54: C26.2, IC6D.+IN, R34.1
- removed net N$55: C29.2, IC6D.-IN, R36.1
- removed net N$56: C19.2, R24.2, R26.1
- removed net N$57: D5.C, IC6A.-IN, R24.1
- removed net N$59: D5.A, IC6A.OUT
- new net N$4: D5.A, R25.1
- new net N$44: C15.2, IC4A.-IN, R24.2, R28.1
- new net N$45: D4.A, R24.1
- new net N$48: C9.1, IC2B.OUT, IC4A.+IN, R10.1, R14.2
- new net N$7: B1.D1, JP2.3
- net +3V3: now also B1.3.3V, B1.AREF, Q1.G, R16.2, R17.2; no longer C15.1, IC2.VO, Q3.G, R31.2, R32.2
- net +5V: now also B1.5V, C1.+, C15.1, C17.2, C18.2, C2.1, C6.2, IC1.VCC, IC2P.V+, IC3P.V+, IC4P.V+, JP3.2, JP4.2, R12.2, R13.2; no longer C13.2, C14.1, C25.2, C27.2, C7.1, C9.+, IC1P.V+, IC2.VI, IC5P.V+, IC6P.V+, ISP.2, JP4.3, JP4.4, L1.2, L2.1, L3.1, R27.2, R28.2, R4.2, U$1.VCC
- net GND: now also B1.GND, B1.GND@0, B1.GND@1, B1.GND@2, C17.1, C5.2, C6.1, IC1.GND, IC2P.V-, IC3P.V-, IC4P.V-, JP2.2, JP2.4, JP3.1; no longer C10.1, C11.1, C12.2, C13.1, C14.2, C15.2, C16.2, C17.2, C19.1, C25.1, C27.1, C3.2, C4.2, C7.2, C8.2, C9.-, IC1P.V-, IC2.GND, IC3.AGND, IC3.GND@1, IC3.GND@2, IC5P.V-, IC6P.V-, ISP.10, ISP.8, JP2.GND, JP4.2, U$1.GND
- net GND1: now also C11.1, C12.1, C5.1, IC1.VO, IC2A.+IN, IC2D.+IN, R20.2, R21.2, R26.2, R27.2; no longer C17.1, C20.1, C21.1, C24.1, C26.1, IC1A.+IN, IC1D.+IN, IC5B.+IN, IC6B.+IN, R29.2, R30.2, R35.2, R36.2, U$1.VO
- net L_NEEDLE: now also B1.A0, IC3B.OUT, R30.1; no longer C28.1, IC3.PC1(ADC1/PCINT9), IC5D.OUT, R14.2
- net L_PEAK: now also B1.A2, R29.2; no longer IC3.PC0(ADC0/PCINT8), R25.2
- net N$1: now also IC3B.-IN, R26.1, R30.2; no longer IC5B.-IN, R13.1, R14.1, R15.1, R19.2
- net N$10: now also C13.2, IC3A.OUT, IC3B.+IN, R22.2; no longer C22.2, IC5C.-IN, R29.1
- net N$11: now also C16.2, IC4B.-IN, R25.2, R29.1; no longer C18.2, R23.2, R25.1
- net N$13: now also IC3C.-IN, R27.1, R31.2; no longer C22.1, IC5C.OUT, R13.2, R33.2
- net N$14: now also C11.2, IC3A.+IN, R18.1; no longer C24.2, IC5D.+IN, R33.1
- net N$15: now also IC3A.-IN, R20.1, R22.1; no longer C28.2, IC5D.-IN, R35.1
- net N$16: now also D2.C, R5.1, R8.2; no longer D2.A, R6.1, R9.2
- net N$17: now also C12.2, IC3D.+IN, R19.1; no longer D4.A, IC5A.OUT
- net N$18: now also C3.2; no longer C5.2
- net N$19: now also C7.1, IC2A.-IN, R4.2; no longer C31.1, IC1A.-IN, R6.2
- net N$2: now also B1.D0, JP2.1; no longer C10.2, IC3.PB6(XTAL1/TOSC1/PCINT6), Q1.2
- net N$20: now also D4.C, IC4A.OUT; no longer C3.1, JP2.VBUS, L2.2
- net N$23: now also IC3D.-IN, R21.1, R23.1; no longer IC3.PB4(MISO/PCINT4), ISP.9
- net N$24: now also C14.1, R15.1, R19.2; no longer IC3.PC6(/RESET/PCINT14), ISP.5, R4.1
- net N$25: now also C7.2, D2.A, IC2B.+IN, R4.1; no longer C31.2, D2.C, IC1B.+IN, R5.1
- net N$26: now also IC2A.OUT; no longer IC1A.OUT
- net N$27: now also C9.2, IC2B.-IN, R10.2, R8.1; no longer C30.2, IC1B.-IN, R11.2, R9.1
- net N$28: now also C14.2, IC3C.+IN, IC3D.OUT, R23.2; no longer C12.1, IC3.AREF
- net N$3: now also B1.SDA, Q1.D, R12.1; no longer IC3.PC4(ADC4/SDA/PCINT12), Q2.D, R27.1
- net N$31: now also D3.C, R7.1, R9.2; no longer D3.A, R10.2, R8.1
- net N$33: now also C8.1, IC2D.-IN, R6.2; no longer C33.1, IC1D.-IN, R8.2
- net N$34: now also C8.2, D3.A, IC2C.+IN, R6.1; no longer C33.2, D3.C, IC1C.+IN, R7.1
- net N$35: now also IC2D.OUT; no longer IC1D.OUT
- net N$36: now also C10.2, IC2C.-IN, R11.2, R9.1; no longer C32.2, IC1C.-IN, R10.1, R12.2
- net N$37: now also C10.1, IC2C.OUT, IC4B.+IN; no longer C30.1, IC1B.OUT, IC5A.+IN
- net N$38: now also C4.2; no longer C6.2
- net N$39: now also C4.1; no longer C6.1
- net N$40: now also C3.1; no longer C5.1
- net N$6: now also B1.SCL, Q2.D, R13.1; no longer IC3.PC5(ADC5/SCL/PCINT13), Q3.D, R28.1
- net N$8: now also D5.C, IC4B.OUT; no longer IC5B.OUT, R19.1, R21.2
- net N$9: now also C13.1, R14.1, R18.2; no longer C20.2, IC5C.+IN, R21.1
- net R_NEEDLE: now also B1.A1, IC3C.OUT, R31.1; no longer C29.1, IC3.PC2(ADC2/PCINT10), IC6D.OUT, R17.2
- net R_PEAK: now also B1.A3, R28.2; no longer IC3.PC3(ADC3/PCINT11), R26.2
- net SCL: now also JP3.3, JP4.3, Q2.S, R17.1; no longer JP4.5, JP4.6, Q3.S, R32.1
- net SDA: now also JP3.4, JP4.4, Q1.S, R16.1; no longer JP4.7, JP4.8, Q2.S, R31.1
Other:
- note removed: "*) as close to USB as possible"
- note removed: "*) ceramic"
- moved on the sheet: C1, C10, C11, C12, C13, C14, C15, C16, C17, C18, C2, C3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
