File: hardware/vu_meter_2.sch (EAGLE design)
At the start: 64 parts, among them IC1 MCP1525, IC2 MCP604, IC3 MCP6004, IC4 MCP6002SN, Q1 BSS138, Q2 BSS138

Commit message: Added hardware documentation
Parts:
- removed B1: ARDUINO_UNO_R3NO_HOLES, SparkFun-Boards:ARDUINO_UNO_R3NO_HOLES
- removed JP1: AUDIO-JACK2PTH, SparkFun:AUDIO-JACK2PTH
- removed JP2: (no value), pinhead:PINHD-2X2
- removed JP3, JP4: (no value), pinhead:PINHD-1X4
- added C19: 22pF, rcl:C-EUC0805
- added C20: 10uF, rcl:C-EUC0805
- added C21: 220pF, rcl:C-EUC0805
- added C22: 47nF, rcl:C-EUC0805
- added C23: 1uF, rcl:C-EUC0805
- added C24: 220nF, rcl:C-EUC0805
- added C25: 33pF, rcl:C-EUC0805
- added C26, C27, C28, C30, C33, C34: 100nF, rcl:C-EUC0805
- added C29, C31: 100uF, rcl:CPOL-EUB/3528-21R
- added C32: 10uF, rcl:CPOL-EUB/3528-21R
- added D1: BAS70-04, diode:BAS70-04
- added D6: BAT85, diode:DIODE-MINIMELF
- added H1, H2, H3, H4: MOUNT-HOLE3.2, holes:MOUNT-HOLE3.2
- added IC5: MEGA88, avr-7:MEGA48/88/168-AU
- added IC6: MCP1700 3V3, linear:MCP1703CB
- added IC7: REG1117, burr-brown:REG1117
- added J1: 455-1750-1-ND, SparkFun-Connectors:CONN_03
- added J2: (no value), SparkFun-Connectors:CONN_02
- added J3: (no value), SparkFun-Connectors:CONN_03X22X3_SILK_MALE_PTH
- added J4: (no value), SparkFun-Connectors:CONN_04X2
- added L1: 10uH, rcl:L-EUL3216C
- added Q3: (no value), crystal:CRYSTALHC49S
- added R32: 220, rcl:R-EU_R0805
- added R33: 1k, rcl:R-EU_R0805
- added R34: 220k, rcl:R-EU_R0805
- added R35: 22k, rcl:R-EU_R0805
- added R36: 10k, rcl:R-TRIMM3296W
- added R37: 10k, rcl:R-EU_R0805
- C1: value 100uF -> 22pF; device rcl:CPOL-EUB/3528-21R -> rcl:C-EUC0805
- C10: value 22pF -> 330n
- C11, C12: value 330n -> 330nF
- C14: value 330n -> 100nF
- C16: value 47nF -> 470nF
- C17: value 100nF -> 220pF
- C3: value 220nF -> 470nF
- C5: value 1uF* -> 1uF; TYPE (none) -> ceramic
- C7, C9: value 22pF -> 220pF
- C8: value 22pF -> 33pF
- D2: value BAT54S -> 1N4148; device diode:BAV199 -> diode:DIODE-MINIMELF
- D3: value BAT54S -> BAS70-04; device diode:BAV199 -> diode:BAS70-04
- D4: device diode:BAT60J -> diode:DIODE-MINIMELF
- D5: value 1N4148 -> BAT85; device diode:BAT60J -> diode:DIODE-MINIMELF
- IC2: value MCP604 -> MCP6004
- IC3: value MCP6004 -> MCP604SL
- IC4: value MCP6002SN -> MCP6004; device linear:MCP602SN -> linear:MCP604SL
- R1: value 10k -> 220k; device vu_meter:POT1 -> rcl:R-EU_R0805
- R10, R2, R4, R5, R8: value 100k -> 10k
- R11: value 100k -> 220k
- R15: device rcl:R-EU_M0805 -> rcl:R-EU_R0805
- R19, R21: value 220k -> 10k
- R23: value 82k -> 10k
- R25: value 220 -> 10k
- R26: value 30k -> 47k
- R27: value 30k -> 10k; device rcl:R-EU_M0805 -> rcl:R-EU_R0805
- R29: value 1k -> 82k
- R3: value 100k -> 22k
- R31: value 220k -> 47k
- R6: value 100k -> 10k; device rcl:R-EU_R0805 -> rcl:R-TRIMM3296W
- R7, R9: value 100k -> 220k; device rcl:R-EU_R0805 -> rcl:R-EU_M0805
Connections:
- removed net N$3: B1.SDA, Q1.D, R12.1
- removed net N$6: B1.SCL, Q2.D, R13.1
- new net IN: J1.3, R6.E
- new net IN1: J1.1, R36.E
- new net N$12: D3.C2, R21.1, R27.2
- new net N$21: D3.C1A2, IC3C.OUT
- new net N$22: C17.2, IC4C.-IN, R25.2, R27.1
- new net N$29: C10.2, IC4A.+IN, IC4B.OUT, R29.2
- new net N$30: C22.2, IC3D.-IN, R32.2, R33.1
- new net N$32: C17.1, IC3D.+IN, IC4C.OUT, R25.1, R9.2
- new net N$39: IC5.PB3(MOSI/OC2A/PCINT3), J3.4
- new net N$43: IC5.PC6(/RESET/PCINT14), J3.5, R37.1
- new net N$47: C32.+, IC7.VIN, J2.2
- new net SCL1: IC5.PC5(ADC5/SCL/PCINT13), Q2.D, R13.1
- new net SDA1: IC5.PC4(ADC4/SDA/PCINT12), Q1.D, R12.1
- new net VCC: C26.1, C27.1, C29.+, IC5.VCC@1, IC5.VCC@2, J4.3, J4.4, L1.1, R12.2, R13.2, R37.2
- net +3V3: now also C15.1, C20.1, C22.1, C30.1, C33.2, C34.2, IC5.AREF, IC6.VO; no longer B1.3.3V, B1.AREF
- net +5V: now also C14.2, C23.1, C28.1, C31.+, D5.C, D6.C, IC5.AVCC, IC6.VI, IC7.VOUT, J3.2, L1.2; no longer B1.5V, C1.+, C15.1, C16.1, C17.2, JP3.2, JP4.2, R12.2, R13.2
- net GND: now also C1.1, C14.1, C19.1, C20.2, C23.2, C26.2, C27.2, C28.2, C29.-, C30.2, C31.-, C32.-, C33.1, C34.1, IC5.AGND, IC5.GND@1, IC5.GND@2, IC6.GND, IC7.GND, J1.2, J2.1, J3.6, J4.1, J4.2, R36.A, R6.A; no longer B1.GND, B1.GND@0, B1.GND@1, B1.GND@2, C1.-, C17.1, JP1.RSH, JP1.SLEEVE, JP1.TSH, JP2.2, JP2.4, JP3.1, JP4.1, R1A.A-1, R1B.A-1
- net GND1: now also IC3B.+IN, IC3C.+IN, IC4D.+IN, R11.2, R31.2; no longer IC2D.+IN, R21.2, R27.2
- net L_NEEDLE: now also IC2D.OUT, IC5.PC0(ADC0/PCINT8); no longer B1.A0, IC3B.OUT
- net L_PEAK: now also IC5.PC2(ADC2/PCINT10), R28.2; no longer B1.A2, R29.2
- net N$1: now also IC2D.-IN; no longer IC3B.-IN
- net N$10: now also IC2C.OUT, IC2D.+IN; no longer IC3A.OUT, IC3B.+IN
- net N$11: now also R11.1; no longer C16.2, R25.2
- net N$13: now also C21.1, R19.2, R21.2, R23.1; no longer R27.1, R31.2
- net N$14: now also IC2C.+IN; no longer IC3A.+IN
- net N$15: now also IC2C.-IN; no longer IC3A.-IN
- net N$16: now also D1.C2; no longer D2.C
- net N$17: now also C21.2, D3.A1, IC4C.+IN; no longer C12.2, IC3D.+IN
- net N$18: now also C8.2, IC2A.OUT, R1.1; no longer R1B.S-2
- net N$19: now also IC3B.-IN; no longer IC2A.-IN
- net N$2: now also IC4A.-IN, R31.1, R7.2; no longer B1.D0, JP2.1
- net N$20: now also D2.C, IC3A.OUT; no longer D4.C, IC4A.OUT
- net N$23: now also C16.2, C25.2, IC4D.OUT, R34.1; no longer IC3D.-IN, R21.1, R23.1
- net N$24: now also C16.1, R23.2; no longer C14.1, R15.1, R19.2
- net N$25: now also D1.A1; no longer D2.A
- net N$26: now also D1.C1A2, IC3B.OUT; no longer D2.AC, IC2A.OUT
- net N$28: now also C10.1, R15.2, R9.1; no longer C14.2, IC3C.+IN, IC3D.OUT, R23.2
- net N$31: now also D4.A, R32.1; no longer D3.C, R7.1, R9.2
- net N$33: now also D4.C, IC3D.OUT; no longer C8.1, IC2D.-IN, R3.1, R6.2, R7.2
- net N$34: now also C25.1, D6.A, IC4D.-IN, R34.2, R35.1; no longer C8.2, D3.A, IC2C.+IN, R6.1
- net N$35: now also C24.1, R35.2; no longer D3.AC, IC2D.OUT
- net N$36: now also C24.2, R36.S; no longer C10.2, IC2C.-IN, R11.2, R9.1
- net N$37: now also C19.2, IC5.PB6(XTAL1/TOSC1/PCINT6), Q3.2; no longer C10.1, IC2C.OUT, IC4B.+IN, R11.1, R15.2
- net N$38: now also C1.2, IC5.PB7(XTAL2/TOSC2/PCINT7), Q3.1; no longer C4.2, R1A.S-2
- net N$4: now also C8.1, IC2A.-IN, R1.2, R3.1; no longer R25.1
- net N$41: now also IC5.PB5(SCK/PCINT5), J3.3; no longer JP1.RING, R1B.E-3
- net N$42: now also IC5.PB4(MISO/PCINT4), J3.1; no longer JP1.TIP, R1A.E-3
- net N$44: now also IC3A.-IN; no longer IC4A.-IN
- net N$45: now also D2.A; no longer D4.A
- net N$48: now also IC3A.+IN; no longer IC4A.+IN
- net N$7: now also C12.2, IC4B.+IN, R15.1; no longer B1.D1, JP2.3
- net N$8: now also C4.2, R6.S; no longer D5.C, IC4B.OUT
- net R_NEEDLE: now also IC4A.OUT, IC5.PC1(ADC1/PCINT9), R7.1; no longer B1.A1, IC3C.OUT, R31.1
- net R_PEAK: now also IC5.PC3(ADC3/PCINT11), R33.2; no longer B1.A3, R28.2
- net SCL: now also J4.5, J4.6; no longer JP3.3, JP4.3
- net SDA: now also J4.7, J4.8; no longer JP3.4, JP4.4
Other:
- moved on the sheet: C10, C11, C12, C13, C14, C15, C16, C17, C18, C2, C3, C4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
